Commit message: change blue

File: src/demo_diff_drive_pkg/description/robot_core.xacro (robot description, xacro)
@@ -39,5 +39,5 @@
     </link>
     <gazebo reference="chassis_link">
-        <material>Gazebo/Blue</material>
+        <material>Gazebo/SkyBlue</material>
     </gazebo>
     <!-- left wheel link -->

Commit message: change car color

File: src/demo_diff_drive_pkg/description/robot_core.xacro (robot description, xacro)
@@ -39,5 +39,5 @@
     </link>
     <gazebo reference="chassis_link">
-        <material>Gazebo/SkyBlue</material>
+        <material>Gazebo/Orange</material>
     </gazebo>
     <!-- left wheel link -->
